File: inclinometer-breakout-SCA100T.brd (EAGLE design)
At the start: 100 x 80 mm, 8 parts

Commit message: updated files
Parts:
- removed J1: (no value), SparkFun-Connectors:1X08_ROUND
- added JP1, JP2, JP3, JP4: STAND-OFF, SparkFun:STAND-OFF
- added X1: (no value), con-phoenix-254:8POL254
- moved LOGO1 63.9 mm to (29.8, 13.3)
- moved C3 55.3 mm to (24.1, 11.4)
- moved R2 53.1 mm to (26.2, 7.62), turned to 90 degrees
- moved C1 50.6 mm to (24.8, 14.6), turned to 270 degrees
- moved R1 50.2 mm to (24.1, 7.62), turned to 90 degrees
- moved C2 49.8 mm to (22.9, 14.6), turned to 270 degrees
- moved U$1 34.0 mm to (8.64, 15.4)
Connections:
- net CS: now also X1.1; no longer J1.3
- net GND: now also X1.8; no longer J1.7
- net MISO: now also X1.3; no longer J1.5
- net MOSI: now also X1.2; no longer J1.6
- net SCK: now also X1.4; no longer J1.4
- net VDD: now also X1.7; no longer J1.8
- net VOUT_X: now also X1.6; no longer J1.1
- net VOUT_Y: now also X1.5; no longer J1.2
Routing:
- net GND: track 0.00 -> 54.7 mm
- net VOUT_Y: track 0.00 -> 36.1 mm
- net CS: track 0.00 -> 29.2 mm
- net VOUT_X: track 0.00 -> 25.0 mm
- net N$2: track 0.00 -> 21.4 mm
- net MOSI: track 0.00 -> 15.3 mm
- net MISO: track 0.00 -> 14.0 mm
- net VDD: track 0.00 -> 12.5 mm
- net SCK: track 0.00 -> 8.92 mm
- net N$1: track 0.00 -> 8.04 mm
Other:
- board size 100 x 80 mm -> 33.1 x 24.1 mm
