File: inclinometer-breakout-SCA100T.sch (EAGLE design)
At the start: 8 parts

Commit message: updated files
Parts:
- removed J1: (no value), SparkFun-Connectors:M08
- added X1: (no value), con-phoenix-254:MPT8
Connections:
- net CS: now also X1-1.1; no longer J1.3
- net GND: now also X1-8.1; no longer J1.7
- net MISO: now also X1-3.1; no longer J1.5
- net MOSI: now also X1-2.1; no longer J1.6
- net SCK: now also X1-4.1; no longer J1.4
- net VDD: now also X1-7.1; no longer J1.8
- net VOUT_X: now also X1-6.1; no longer J1.1
- net VOUT_Y: now also X1-5.1; no longer J1.2
Changed lines of the file:
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@@
 <part name="GND4" library="SparkFun-Aesthetics" deviceset="GND" device=""/>
 <part name="LOGO1" library="SparkFun-Aesthetics" deviceset="OSHW-LOGO" device="M"/>
-<part name="J1" library="SparkFun-Connectors" deviceset="M08" device=""/>
-<part name="GND5" library="SparkFun-Aesthetics" deviceset="GND" device=""/>
-<part name="SUPPLY1" library="SparkFun-Aesthetics" deviceset="VDD" device=""/>
 <part name="SUPPLY2" library="SparkFun-Aesthetics" deviceset="VDD" device=""/>
+<part name="GND6" library="SparkFun-Aesthetics" deviceset="GND" device=""/>
+<part name="SUPPLY3" library="SparkFun-Aesthetics" deviceset="VDD" device=""/>
+<part name="X1" library="con-phoenix-254" deviceset="MPT8" device=""/>
 </parts>
 <sheets>
@@
 <instance part="GND4" gate="1" x="20.32" y="10.16"/>
 <instance part="LOGO1" gate="G$1" x="22.86" y="45.72"/>
-<instance part="J1" gate="G$1" x="53.34" y="50.8"/>
-<instance part="GND5" gate="1" x="81.28" y="53.34"/>
-<instance part="SUPPLY1" gate="VDD" x="81.28" y="63.5"/>
 <instance part="SUPPLY2" gate="VDD" x="99.06" y="25.4"/>
+<instance part="GND6" gate="1" x="76.2" y="40.64"/>
+<instance part="SUPPLY3" gate="VDD" x="76.2" y="48.26"/>
+<instance part="X1" gate="-1" x="53.34" y="78.74" rot="MR0"/>
+<instance part="X1" gate="-2" x="53.34" y="73.66" rot="MR0"/>
+<instance part="X1" gate="-3" x="53.34" y="68.58" rot="MR0"/>
+<instance part="X1" gate="-4" x="53.34" y="63.5" rot="MR0"/>
+<instance part="X1" gate="-5" x="53.34" y="58.42" rot="MR0"/>
+<instance part="X1" gate="-6" x="53.34" y="53.34" rot="MR0"/>
+<instance part="X1" gate="-7" x="53.34" y="48.26" rot="MR0"/>
+<instance part="X1" gate="-8" x="53.34" y="43.18" rot="MR0"/>
 </instances>
 <busses>
@@
 </segment>
 <segment>
-<pinref part="J1" gate="G$1" pin="1"/>
-<wire x1="58.42" y1="43.18" x2="71.12" y2="43.18" width="0.1524" layer="91"/>
-<label x="63.5" y="43.18" size="1.778" layer="95"/>
+<wire x1="55.88" y1="53.34" x2="71.12" y2="53.34" width="0.1524" layer="91"/>
+<label x="60.96" y="53.34" size="1.778" layer="95"/>
+<pinref part="X1" gate="-6" pin="1"/>
 </segment>
 </net>
@@
 </segment>
 <segment>
-<pinref part="J1" gate="G$1" pin="2"/>
-<wire x1="58.42" y1="45.72" x2="71.12" y2="45.72" width="0.1524" layer="91"/>
-<label x="63.5" y="45.72" size="1.778" layer="95"/>
+<wire x1="55.88" y1="58.42" x2="68.58" y2="58.42" width="0.1524" layer="91"/>
+<label x="60.96" y="58.42" size="1.778" layer="95"/>
+<pinref part="X1" gate="-5" pin="1"/>
 </segment>
 </net>
@@
 </segment>
 <segment>
-<pinref part="J1" gate="G$1" pin="7"/>
-<wire x1="58.42" y1="58.42" x2="81.28" y2="58.42" width="0.1524" layer="91"/>
-<label x="63.5" y="58.42" size="1.778" layer="95"/>
-<wire x1="81.28" y1="58.42" x2="81.28" y2="55.88" width="0.1524" layer="91"/>
-<pinref part="GND5" gate="1" pin="GND"/>
+<wire x1="55.88" y1="43.18" x2="76.2" y2="43.18" width="0.1524" layer="91"/>
+<label x="60.96" y="43.18" size="1.778" layer="95"/>
+<pinref part="GND6" gate="1" pin="GND"/>
+<pinref part="X1" gate="-8" pin="1"/>
 </segment>
 </net>
@@
 </segment>
 <segment>
-<pinref part="J1" gate="G$1" pin="3"/>
-<wire x1="58.42" y1="48.26" x2="71.12" y2="48.26" width="0.1524" layer="91"/>
-<label x="63.5" y="48.26" size="1.778" layer="95"/>
+<wire x1="55.88" y1="78.74" x2="66.04" y2="78.74" width="0.1524" layer="91"/>
+<label x="60.96" y="78.74" size="1.778" layer="95"/>
+<pinref part="X1" gate="-1" pin="1"/>
 </segment>
 </net>
@@
 </segment>
 <segment>
-<pinref part="J1" gate="G$1" pin="6"/>
-<wire x1="58.42" y1="55.88" x2="71.12" y2="55.88" width="0.1524" layer="91"/>
-<label x="63.5" y="55.88" size="1.778" layer="95"/>
+<wire x1="55.88" y1="73.66" x2="68.58" y2="73.66" width="0.1524" layer="91"/>
+<label x="60.96" y="73.66" size="1.778" layer="95"/>
+<pinref part="X1" gate="-2" pin="1"/>
 </segment>
 </net>
@@
 </segment>
 <segment>
-<pinref part="J1" gate="G$1" pin="5"/>
-<wire x1="58.42" y1="53.34" x2="71.12" y2="53.34" width="0.1524" layer="91"/>
-<label x="63.5" y="53.34" size="1.778" layer="95"/>
+<wire x1="55.88" y1="68.58" x2="68.58" y2="68.58" width="0.1524" layer="91"/>
+<label x="60.96" y="68.58" size="1.778" layer="95"/>
+<pinref part="X1" gate="-3" pin="1"/>
 </segment>
 </net>
@@
 </segment>
 <segment>
-<pinref part="J1" gate="G$1" pin="4"/>
-<wire x1="58.42" y1="50.8" x2="71.12" y2="50.8" width="0.1524" layer="91"/>
-<label x="63.5" y="50.8" size="1.778" layer="95"/>
+<wire x1="55.88" y1="63.5" x2="68.58" y2="63.5" width="0.1524" layer="91"/>
+<label x="60.96" y="63.5" size="1.778" layer="95"/>
+<pinref part="X1" gate="-4" pin="1"/>
 </segment>
 </net>
 <net name="VDD" class="0">
-<segment>
-<pinref part="J1" gate="G$1" pin="8"/>
-<wire x1="58.42" y1="60.96" x2="81.28" y2="60.96" width="0.1524" layer="91"/>
-<label x="63.5" y="60.96" size="1.778" layer="95"/>
-<wire x1="81.28" y1="60.96" x2="81.28" y2="63.5" width="0.1524" layer="91"/>
-<pinref part="SUPPLY1" gate="VDD" pin="VDD"/>
-</segment>
 <segment>
 <pinref part="U$1" gate="G$1" pin="VDD"/>
@@
 <label x="50.8" y="25.4" size="1.778" layer="95"/>
 </segment>
+<segment>
+<label x="60.96" y="48.26" size="1.778" layer="95"/>
+<wire x1="55.88" y1="48.26" x2="76.2" y2="48.26" width="0.1524" layer="91"/>
+<pinref part="SUPPLY3" gate="VDD" pin="VDD"/>
+<pinref part="X1" gate="-7" pin="1"/>
+</segment>
 </net>
